File: Test0805.kicad_pcb (KiCad board)
At the start: 2 copper layers, 27.9 x 15.2 mm, 7 parts

Commit message: Add indication of polarity.
Other:
- board text added: "+"
Changed lines of the file:
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@@
     (links 8)
     (no_connects 0)
-    (area 0 0 0 0)
+    (area 126.924999 100.45 155.015001 118.09)
     (thickness 1.6)
-    (drawings 6)
+    (drawings 7)
     (tracks 23)
     (zones 0)
@@
     )
   )
+  (gr_text + (at 130.81 109.22) (layer B.SilkS)
+    (effects (font (size 1.5 1.5) (thickness 0.3)) (justify mirror))
+  )
   (gr_arc (start 147.32 109.22) (end 147.32 101.6) (angle 90) (layer Edge.Cuts) (width 0.15))
